Commit message: wip:add arm

File: showcase/robot-arm/public/kuka/urdf/unnamed.urdf (robot description, URDF)
Before this commit: robot unnamed, 6 links, 5 joints
Links:
- added link end_effector_link; visual box size=1.0 1.0 1.0
- link kuka-arm-000_link: geometry visual mesh filename=../meshes/stl/kuka-arm-000.stl scale=2 2 2
- link kuka-arm-001_link: geometry visual mesh filename=../meshes/stl/kuka-arm-001.stl scale=2 2 2
- link kuka-arm-002_link: geometry visual mesh filename=../meshes/stl/kuka-arm-002.stl scale=2 2 2
- link kuka-arm-003_link: geometry visual mesh filename=../meshes/stl/kuka-arm-003.stl scale=2 2 2
- link kuka-arm-004_link: geometry visual mesh filename=../meshes/stl/kuka-arm-004.stl scale=2 2 2
- link kuka-arm-005_link: geometry visual mesh filename=../meshes/stl/kuka-arm-005.stl scale=2 2 2
Joints:
- added joint end_effector_joint: type fixed, parent kuka-arm-000_link, child end_effector_link, origin xyz=-2.99080 0.06848 0.07536 rpy=0.00000 0.00000 0.00000
- joint kuka-arm-000_link_joint: limit lower=-1.00000 upper=1.00000 effort=0.00000 velocity=0.00000 -> lower=-1.57080 upper=1.57080 effort=0.00000 velocity=0.00000; origin xyz=6.29044 -0.19594 0.07072 rpy=0.00000 0.00000 -0.00000 -> xyz=12.58088 -0.39188 0.14144 rpy=0.00000 0.00000 -0.00000
- joint kuka-arm-001_link_joint: limit lower=-0.33000 upper=0.49000 effort=1.11000 velocity=0.00000 -> lower=-1.57080 upper=1.57080 effort=1.11000 velocity=0.00000; origin xyz=16.66716 0.08146 -0.95556 rpy=-0.00000 0.00000 -0.00000 -> xyz=33.33432 0.16292 -1.91112 rpy=-0.00000 0.00000 -0.00000
- joint kuka-arm-002_link_joint: limit lower=-0.33000 upper=0.49000 effort=1.11000 velocity=0.00000 -> lower=-1.57080 upper=1.57080 effort=1.11000 velocity=0.00000; origin xyz=0.01569 -0.13262 21.69338 rpy=0.00000 -0.00000 0.00000 -> xyz=0.03138 -0.26524 43.38676 rpy=0.00000 -0.00000 0.00000
- joint kuka-arm-003_link_joint: limit lower=-0.33000 upper=0.49000 effort=1.11000 velocity=0.00000 -> lower=-1.57080 upper=1.57080 effort=1.11000 velocity=0.00000; origin xyz=8.21240 0.22730 6.83013 rpy=-0.00000 -0.00000 -0.00000 -> xyz=16.42480 0.45460 13.66026 rpy=-0.00000 -0.00000 -0.00000
- joint kuka-arm-004_link_joint: limit lower=-1.00000 upper=1.00000 effort=1.11000 velocity=0.00000 -> lower=-2.96706 upper=2.96706 effort=1.11000 velocity=0.00000; origin xyz=0.00971 -0.01443 9.84568 rpy=0.00000 0.00000 0.00000 -> xyz=0.01942 -0.02886 19.69136 rpy=0.00000 0.00000 0.00000

Commit message: consider constraints

File: showcase/robot-arm/public/kuka/urdf/unnamed.urdf (robot description, URDF)
Before this commit: robot unnamed, 7 links, 6 joints
Links:
- removed link end_effector_link
- added link kuka-arm-000-2_link; visual mesh filename=../meshes/stl/Cylinder.003.stl scale=1 1 1
- link kuka-arm-000_link: geometry visual mesh filename=../meshes/stl/kuka-arm-000.stl scale=1 1 1
- link kuka-arm-001_link: geometry collision cylinder length=18123.28516 radius=6178.39258; visual mesh filename=../meshes/stl/kuka-arm-001.stl scale=1 1 1
- link kuka-arm-002_link: geometry visual mesh filename=../meshes/stl/kuka-arm-002.stl scale=1 1 1
- link kuka-arm-003_link: geometry visual mesh filename=../meshes/stl/kuka-arm-003.stl scale=1 1 1
- link kuka-arm-004_link: geometry visual mesh filename=../meshes/stl/kuka-arm-004.stl scale=1 1 1
- link kuka-arm-005_link: geometry visual mesh filename=../meshes/stl/kuka-arm-005.stl scale=1 1 1
Joints:
- removed joint end_effector_joint
- added joint kuka-arm-000-2_link_joint: type revolute, parent kuka-arm-000_link, child kuka-arm-000-2_link, origin xyz=0.59303 0.13547 -7.77616 rpy=0.00000 0.00000 0.00000, axis 0.00000 0.00000 1.00000, limit lower=0.00000 upper=1.00000 effort=0.00000 velocity=0.00000
- joint kuka-arm-000_link_joint: limit lower=-1.57080 upper=1.57080 effort=0.00000 velocity=0.00000 -> lower=0.00000 upper=0.00000 effort=0.00000 velocity=0.00000; origin xyz=12.58088 -0.39188 0.14144 rpy=0.00000 0.00000 -0.00000 -> xyz=6.29044 -0.19594 0.07072 rpy=0.00000 0.00000 -0.00000
- joint kuka-arm-001_link_joint: limit lower=-1.57080 upper=1.57080 effort=1.11000 velocity=0.00000 -> lower=-0.33000 upper=0.49000 effort=1.11000 velocity=0.00000; origin xyz=33.33432 0.16292 -1.91112 rpy=-0.00000 0.00000 -0.00000 -> xyz=16.66716 0.08146 -0.95556 rpy=-0.00000 0.00000 -0.00000
- joint kuka-arm-002_link_joint: limit lower=-1.57080 upper=1.57080 effort=1.11000 velocity=0.00000 -> lower=-0.33000 upper=0.49000 effort=1.11000 velocity=0.00000; origin xyz=0.03138 -0.26524 43.38676 rpy=0.00000 -0.00000 0.00000 -> xyz=0.01569 -0.13262 21.69338 rpy=0.00000 -0.00000 0.00000
- joint kuka-arm-003_link_joint: limit lower=-1.57080 upper=1.57080 effort=1.11000 velocity=0.00000 -> lower=-0.33000 upper=0.49000 effort=1.11000 velocity=0.00000; origin xyz=16.42480 0.45460 13.66026 rpy=-0.00000 -0.00000 -0.00000 -> xyz=8.21240 0.22730 6.83013 rpy=-0.00000 -0.00000 -0.00000
- joint kuka-arm-004_link_joint: limit lower=-2.96706 upper=2.96706 effort=1.11000 velocity=0.00000 -> lower=-1.00000 upper=1.00000 effort=1.11000 velocity=0.00000; origin xyz=0.01942 -0.02886 19.69136 rpy=0.00000 0.00000 0.00000 -> xyz=0.00971 -0.01443 9.84568 rpy=0.00000 0.00000 0.00000
